Commit message: first commit

File: ffw_description/ros2_control/ffw_a3/ffw_a3.ros2_control.xacro (robot description, xacro)
@@ -1,5 +1,5 @@
 <?xml version="1.0"?>
 <robot xmlns:xacro="http://www.ros.org/wiki/xacro">
-  <xacro:macro name="ffw_a3_system" params="use_sim:=^|false use_mock_hardware:=^|false mock_sensor_commands:=^|false">
+  <xacro:macro name="ffw_a3_system" params="use_sim:=^|false use_mock_hardware:=^|false port_name:=^|/dev/serial/by-id/usb-ROBOTIS_STM32_Virtual_ComPort_3151388A3434-if00 mock_sensor_commands:=^|false">
     <xacro:property name="initial_positions" value="${load_yaml(initial_positions_file)['initial_positions']}"/>
     <ros2_control name="ffw_a3" type="system" is_async="true">
@@ -18,5 +18,5 @@
           <xacro:unless value="${use_mock_hardware}">
             <plugin>dynamixel_hardware_interface/DynamixelHardware</plugin>
-            <param name="port_name">/dev/leader</param>
+            <param name="port_name">${port_name}</param>
             <param name="baud_rate">4000000</param>
             <param name="dynamixel_model_folder">/param/dxl_model</param>

File: ffw_description/urdf/common/leader/ffw_mini_leader_body.urdf.xacro (robot description, xacro)
@@ -2,5 +2,5 @@
 <robot xmlns:xacro="http://www.ros.org/wiki/xacro">
    <xacro:macro name="ffw_mini_leader_body" params="prefix parent *origin">
-      <xacro:property name="meshes_file_direction" value="package://ffw_description/meshes/ffw_lg2_rev3_leader" />
+      <xacro:property name="meshes_file_direction" value="package://ffw_description/meshes/ffw_a3" />
       <joint name="${prefix}joint" type="prismatic">
          <parent link="${parent}"/>

File: ffw_description/urdf/ffw_a3/ffw_a3.urdf.xacro (robot description, xacro)
@@ -4,4 +4,5 @@
   <xacro:arg name="use_mock_hardware" default="false" />
   <xacro:arg name="mock_sensor_commands" default="false" />
+  <xacro:arg name="port_name" default="/dev/serial/by-id/usb-ROBOTIS_STM32_Virtual_ComPort_3151388A3434-if00" />
   <xacro:arg name="prefix" default="" />
   <xacro:include filename="$(find ffw_description)/urdf/common/leader/ffw_mini_leader_body.urdf.xacro" />
@@ -14,4 +15,5 @@
       use_sim="$(arg use_sim)"
       use_mock_hardware="$(arg use_mock_hardware)"
+      port_name="$(arg port_name)"
       mock_sensor_commands="$(arg mock_sensor_commands)" />
 </robot>
