Commit message: Save local development work

File: ffw_description/ros2_control/ffw_f2_follower/ffw_f2_follower.ros2_control.xacro (robot description, xacro)
@@ -325,10 +325,6 @@
         <param name="Profile Velocity">100</param>
         <param name="Profile Acceleration">50</param>
-        <param name="Max Position Limit">151875</param>
-        <param name="Min Position Limit">-131875</param>
-        <!--
         <param name="Max Position Limit">175980</param>
         <param name="Min Position Limit">-152804</param>
-        -->
       </gpio>
       <gpio name="dxl8">
@@ -506,10 +502,6 @@
         <param name="Profile Velocity">100</param>
         <param name="Profile Acceleration">50</param>
-        <param name="Max Position Limit">131875</param>
-        <param name="Min Position Limit">-151875</param>
-        <!--
         <param name="Max Position Limit">152804</param>
         <param name="Min Position Limit">-175980</param>
-        -->
       </gpio>
       <gpio name="dxl38">

File: ffw_description/ros2_control/ffw_f2_follower/ffw_f2_follower_smooth.ros2_control.xacro (robot description, xacro)
@@ -325,10 +325,6 @@
         <param name="Profile Velocity">300</param>
         <param name="Profile Acceleration">150</param>
-        <param name="Max Position Limit">151875</param>
-        <param name="Min Position Limit">-131875</param>
-        <!--
         <param name="Max Position Limit">175980</param>
         <param name="Min Position Limit">-152804</param>
-        -->
       </gpio>
       <gpio name="dxl8">
@@ -506,10 +502,6 @@
         <param name="Profile Velocity">300</param>
         <param name="Profile Acceleration">150</param>
-        <param name="Max Position Limit">131875</param>
-        <param name="Min Position Limit">-151875</param>
-        <!--
         <param name="Max Position Limit">152804</param>
         <param name="Min Position Limit">-175980</param>
-        -->
       </gpio>
       <gpio name="dxl38">

File: ffw_description/urdf/common/follower/ffw_f_follower_body.xacro (robot description, xacro)
@@ -1,5 +1,5 @@
 <?xml version="1.0" encoding="UTF-8"?>
 <robot xmlns:xacro="http://www.ros.org/wiki/xacro">
-   <xacro:macro name="ffw_f_follower_body" params="prefix parent *origin">
+   <xacro:macro name="ffw_f_follower_body" params="prefix parent arm_joint4_upper:=1.0786 arm_l_joint7_lower:=-1.8201 arm_l_joint7_upper:=1.5804 arm_r_joint7_lower:=-1.5804 arm_r_joint7_upper:=1.8201 *origin">
       <xacro:include filename="$(find ffw_description)/urdf/common/follower/wrist_d401.urdf.xacro" />
       <xacro:include filename="$(find realsense2_description)/urdf/_d455.urdf.xacro" />
@@ -205,5 +205,5 @@
          <origin xyz="0.0410041 0.0007 -0.1128" rpy="0 0 0" />
          <axis xyz="0 1 0" />
-         <limit velocity="4.8" effort="1000" lower="-2.9361" upper="1.0786" />
+         <limit velocity="4.8" effort="1000" lower="-2.9361" upper="${arm_joint4_upper}" />
          <dynamics damping="0.1" />
       </joint>
@@ -301,5 +301,5 @@
          <origin xyz="-0.00025 -0.0007 -0.0775" rpy="0 0 0" />
          <axis xyz="1 0 0" />
-         <limit velocity="4.8" effort="1000" lower="-1.8201" upper="1.5804" />
+         <limit velocity="4.8" effort="1000" lower="${arm_l_joint7_lower}" upper="${arm_l_joint7_upper}" />
          <dynamics damping="0.1" />
       </joint>
@@ -432,5 +432,5 @@
          <origin xyz="0.0410041 -0.0007 -0.1128" rpy="0 0 0" />
          <axis xyz="0 1 0" />
-         <limit velocity="4.8" effort="1000" lower="-2.9361" upper="1.0786" />
+         <limit velocity="4.8" effort="1000" lower="-2.9361" upper="${arm_joint4_upper}" />
          <dynamics damping="0.1" />
       </joint>
@@ -528,5 +528,5 @@
          <origin xyz="-0.00025 -0.0007 -0.0775" rpy="0 0 0" />
          <axis xyz="1 0 0" />
-         <limit velocity="4.8" effort="1000" lower="-1.5804" upper="1.8201" />
+         <limit velocity="4.8" effort="1000" lower="${arm_r_joint7_lower}" upper="${arm_r_joint7_upper}" />
          <dynamics damping="0.1" />
       </joint>

File: ffw_description/urdf/ffw_f2_follower/ffw_f2_follower.urdf (robot description, URDF)
Before this commit: robot ffw_f2_follower, 40 links, 39 joints
Joints:
- joint arm_l_joint4: limit lower=-2.9361 upper=1.0786 effort=1000 velocity=4.8 -> lower=-2.9361 upper=1.0785802414820915 effort=1000 velocity=4.8
- joint arm_r_joint4: limit lower=-2.9361 upper=1.0786 effort=1000 velocity=4.8 -> lower=-2.9361 upper=1.0785802414820915 effort=1000 velocity=4.8

File: ffw_description/urdf/ffw_f2_follower/ffw_f2_follower.urdf.xacro (robot description, xacro)
@@ -113,5 +113,14 @@
   <!-- Gazebo plugins/sensors -->
   <xacro:ffw_f2_follower_gazebo prefix="$(arg prefix)" />
-  <xacro:ffw_f_follower_body parent="$(arg prefix)base_link" prefix="$(arg prefix)">
+  <!-- F2 J7 limits use the nominal mechanism envelope. The PH42 EEPROM limits
+       include this range by rounding the raw endpoints outward. -->
+  <xacro:ffw_f_follower_body
+    parent="$(arg prefix)base_link"
+    prefix="$(arg prefix)"
+    arm_joint4_upper="1.0785802414820915"
+    arm_l_joint7_lower="-1.8201"
+    arm_l_joint7_upper="1.5804"
+    arm_r_joint7_lower="-1.5804"
+    arm_r_joint7_upper="1.8201">
     <origin xyz="-0.0753807 0 1.407" rpy="0 0 0" />
   </xacro:ffw_f_follower_body>
